Commit message: update base_mount

File: urdf/ur_macro.xacro (robot description, xacro)
@@ -128,4 +128,11 @@
         />
     </xacro:if>
+    <!-- Define color -->
+    <material name="white">
+      <color rgba="1 1 1 1" />
+    </material>
+    <material name="blue">
+      <color rgba="0 0 1 1" />
+    </material>
     <!-- Add URDF transmission elements (for ros_control) -->
     <!--<xacro:ur_arm_transmission prefix="${prefix}" hw_interface="${transmission_hw_interface}" />-->
@@ -255,8 +262,51 @@
       </xacro:cylinder_inertial>
     </link>
+    <!-- Define my_link -->
+    <link name="base_table">
+      <visual>
+        <origin xyz="0 0 0.25" />
+        <geometry>
+          <box size="1.32 0.8 0.5" />
+        </geometry>
+        <material name="white" />
+      </visual>
+      <collision>
+        <origin xyz="0 0 0.25" />
+        <geometry>
+          <box size="1.32 0.8 0.5" />
+        </geometry>
+      </collision>
+    </link>
+    <link name="profile1">
+      <visual>
+      <origin xyz="0 0 0.45" />
+        <geometry>
+          <box size="0.03 0.35 0.9" />
+        </geometry>
+        <material name="blue" />
+      </visual>
+      <collision>
+        <origin xyz="0 0 0.45" />
+        <geometry>
+          <box size="0.03 0.35 0.9" />
+        </geometry>
+      </collision>
+    </link>
+    <!-- Define my joint -->
+    <joint name="{tf_prefix}base_table_joint" type="fixed">
+      <origin xyz="0 0 0" rpy="0 0 0"/>
+      <parent link="${parent}" />
+      <child link="base_table" />
+    </joint>
+    <joint name="${tf_prefix}profile_joint" type="fixed">
+      <origin xyz="0.3 0 0.505" rpy="0 0 0"/>
+      <parent link="base_table" />
+      <child link="profile1" />
+    </joint>
     <!-- base_joint fixes base_link to the environment -->
     <joint name="${tf_prefix}base_joint" type="fixed">
+      <origin xyz="0 0 0.505" rpy="0 0 0"/>
       <xacro:insert_block name="origin" />
-      <parent link="${parent}" />
+      <parent link="base_table" />
       <child link="${tf_prefix}base_link" />
     </joint>

Commit message: add_sensor_gripper

File: urdf/ur_macro.xacro (robot description, xacro)
@@ -44,4 +44,5 @@
   <xacro:include filename="$(find ur_description)/urdf/inc/ur_transmissions.xacro" />
   <xacro:include filename="$(find ur_description)/urdf/inc/ur_common.xacro" />
+  <xacro:property name="gazebo_axis_z" value="0.0" />
   <xacro:macro name="ur_robot" params="
     name
@@ -52,79 +53,12 @@
     kinematics_parameters_file
     physical_parameters_file
-    visual_parameters_file
-    generate_ros2_control_tag:=true
-    transmission_hw_interface:=hardware_interface/PositionJointInterface
-    safety_limits:=false
-    safety_pos_margin:=0.15
-    safety_k_position:=20
-    use_fake_hardware:=false
-    fake_sensor_commands:=false
-    sim_gazebo:=false
-    sim_ignition:=false
-    headless_mode:=false
-    initial_positions:=${dict(shoulder_pan_joint=0.0,shoulder_lift_joint=-1.57,elbow_joint=0.0,wrist_1_joint=-1.57,wrist_2_joint=0.0,wrist_3_joint=0.0)}
-    use_tool_communication:=false
-    tool_voltage:=0
-    tool_parity:=0
-    tool_baud_rate:=115200
-    tool_stop_bits:=1
-    tool_rx_idle_chars:=1.5
-    tool_tx_idle_chars:=3.5
-    tool_device_name:=/tmp/ttyUR
-    tool_tcp_port:=54321
-    robot_ip:=0.0.0.0
-    script_filename:=to_be_filled_by_ur_robot_driver
-    output_recipe_filename:=to_be_filled_by_ur_robot_driver
-    input_recipe_filename:=to_be_filled_by_ur_robot_driver
-    reverse_port:=50001
-    script_sender_port:=50002
-    reverse_ip:=0.0.0.0
-    script_command_port:=50004
-    trajectory_port:=50003
-    non_blocking_read:=true
-    keep_alive_count:=2"
-    >
+    visual_parameters_file generate_ros2_control_tag:=true transmission_hw_interface:=hardware_interface/PositionJointInterface safety_limits:=false safety_pos_margin:=0.15 safety_k_position:=20 use_fake_hardware:=false fake_sensor_commands:=false sim_gazebo:=false sim_ignition:=false headless_mode:=false initial_positions:=${dict(shoulder_pan_joint=0.0,shoulder_lift_joint=-1.57,elbow_joint=0.0,wrist_1_joint=-1.57,wrist_2_joint=0.0,wrist_3_joint=0.0)} use_tool_communication:=false tool_voltage:=0 tool_parity:=0 tool_baud_rate:=115200 tool_stop_bits:=1 tool_rx_idle_chars:=1.5 tool_tx_idle_chars:=3.5 tool_device_name:=/tmp/ttyUR tool_tcp_port:=54321 robot_ip:=0.0.0.0 script_filename:=to_be_filled_by_ur_robot_driver output_recipe_filename:=to_be_filled_by_ur_robot_driver input_recipe_filename:=to_be_filled_by_ur_robot_driver reverse_port:=50001 script_sender_port:=50002 reverse_ip:=0.0.0.0 script_command_port:=50004 trajectory_port:=50003 non_blocking_read:=true keep_alive_count:=2">
     <!-- Load configuration data from the provided .yaml files -->
-    <xacro:read_model_data
-      joint_limits_parameters_file="${joint_limits_parameters_file}"
-      kinematics_parameters_file="${kinematics_parameters_file}"
-      physical_parameters_file="${physical_parameters_file}"
-      visual_parameters_file="${visual_parameters_file}"
-      force_abs_paths="${sim_gazebo or sim_ignition}"/>
+    <xacro:read_model_data joint_limits_parameters_file="${joint_limits_parameters_file}" kinematics_parameters_file="${kinematics_parameters_file}" physical_parameters_file="${physical_parameters_file}" visual_parameters_file="${visual_parameters_file}" force_abs_paths="${sim_gazebo or sim_ignition}"/>
     <xacro:if value="${generate_ros2_control_tag}">
       <!-- ros2 control include -->
       <xacro:include filename="$(find ur_description)/urdf/ur.ros2_control.xacro" />
       <!-- ros2 control instance -->
-      <xacro:ur_ros2_control
-        name="${name}"
-        use_fake_hardware="${use_fake_hardware}"
-        initial_positions="${initial_positions}"
-        fake_sensor_commands="${fake_sensor_commands}"
-        headless_mode="${headless_mode}"
-        sim_gazebo="${sim_gazebo}"
-        sim_ignition="${sim_ignition}"
-        script_filename="${script_filename}"
-        output_recipe_filename="${output_recipe_filename}"
-        input_recipe_filename="${input_recipe_filename}"
-        tf_prefix="${tf_prefix}"
-        hash_kinematics="${kinematics_hash}"
-        robot_ip="${robot_ip}"
-        use_tool_communication="${use_tool_communication}"
-        tool_voltage="${tool_voltage}"
-        tool_parity="${tool_parity}"
-        tool_baud_rate="${tool_baud_rate}"
-        tool_stop_bits="${tool_stop_bits}"
-        tool_rx_idle_chars="${tool_rx_idle_chars}"
-        tool_tx_idle_chars="${tool_tx_idle_chars}"
-        tool_device_name="${tool_device_name}"
-        tool_tcp_port="${tool_tcp_port}"
-        reverse_port="${reverse_port}"
-        script_sender_port="${script_sender_port}"
-        reverse_ip="${reverse_ip}"
-        script_command_port="${script_command_port}"
-        trajectory_port="${trajectory_port}"
-        non_blocking_read="${non_blocking_read}"
-        keep_alive_count="${keep_alive_count}"
-        />
+      <xacro:ur_ros2_control name="${name}" use_fake_hardware="${use_fake_hardware}" initial_positions="${initial_positions}" fake_sensor_commands="${fake_sensor_commands}" headless_mode="${headless_mode}" sim_gazebo="${sim_gazebo}" sim_ignition="${sim_ignition}" script_filename="${script_filename}" output_recipe_filename="${output_recipe_filename}" input_recipe_filename="${input_recipe_filename}" tf_prefix="${tf_prefix}" hash_kinematics="${kinematics_hash}" robot_ip="${robot_ip}" use_tool_communication="${use_tool_communication}" tool_voltage="${tool_voltage}" tool_parity="${tool_parity}" tool_baud_rate="${tool_baud_rate}" tool_stop_bits="${tool_stop_bits}" tool_rx_idle_chars="${tool_rx_idle_chars}" tool_tx_idle_chars="${tool_tx_idle_chars}" tool_device_name="${tool_device_name}" tool_tcp_port="${tool_tcp_port}" reverse_port="${reverse_port}" script_sender_port="${script_sender_port}" reverse_ip="${reverse_ip}" script_command_port="${script_command_port}" trajectory_port="${trajectory_port}" non_blocking_read="${non_blocking_read}" keep_alive_count="${keep_alive_count}" />
     </xacro:if>
     <!-- Define color -->
@@ -135,4 +69,7 @@
       <color rgba="0 0 1 1" />
     </material>
+    <material name="orange">
+      <color rgba="1 0.5 0 0.5" />
+    </material>
     <!-- Add URDF transmission elements (for ros_control) -->
     <!--<xacro:ur_arm_transmission prefix="${prefix}" hw_interface="${transmission_hw_interface}" />-->
@@ -204,12 +141,12 @@
         </geometry>
       </collision>
-      <xacro:cylinder_inertial radius="${forearm_inertia_radius}" length="${forearm_inertia_length}"  mass="${forearm_mass}">
+      <xacro:cylinder_inertial radius="${forearm_inertia_radius}" length="${forearm_inertia_length}" mass="${forearm_mass}">
         <origin xyz="${-0.5 * forearm_inertia_length} 0.0 ${elbow_offset}" rpy="0 ${pi/2} 0" />
       </xacro:cylinder_inertial>
     </link>
     <link name="${tf_prefix}wrist_1_link">
-	  <xacro:get_visual_params name="wrist_1" type="visual_offset"/>
-      <visual>
-      	<origin xyz="0 0 ${visual_params}" rpy="${pi/2} 0 0"/>
+      <xacro:get_visual_params name="wrist_1" type="visual_offset"/>
+      <visual>
+        <origin xyz="0 0 ${visual_params}" rpy="${pi/2} 0 0"/>
         <geometry>
           <xacro:get_mesh name="wrist_1" type="visual"/>
@@ -222,10 +159,10 @@
         </geometry>
       </collision>
-      <xacro:cylinder_inertial radius="${wrist_1_inertia_radius}" length="${wrist_1_inertia_length}"  mass="${wrist_1_mass}">
+      <xacro:cylinder_inertial radius="${wrist_1_inertia_radius}" length="${wrist_1_inertia_length}" mass="${wrist_1_mass}">
         <origin xyz="0 0 0" rpy="0 0 0" />
       </xacro:cylinder_inertial>
     </link>
     <link name="${tf_prefix}wrist_2_link">
-	  <xacro:get_visual_params name="wrist_2" type="visual_offset"/>
+      <xacro:get_visual_params name="wrist_2" type="visual_offset"/>
       <visual>
         <origin xyz="0 0 ${visual_params}" rpy="0 0 0"/>
@@ -240,10 +177,10 @@
         </geometry>
       </collision>
-      <xacro:cylinder_inertial radius="${wrist_2_inertia_radius}" length="${wrist_2_inertia_length}"  mass="${wrist_2_mass}">
+      <xacro:cylinder_inertial radius="${wrist_2_inertia_radius}" length="${wrist_2_inertia_length}" mass="${wrist_2_mass}">
         <origin xyz="0 0 0" rpy="0 0 0" />
       </xacro:cylinder_inertial>
     </link>
     <link name="${tf_prefix}wrist_3_link">
-	  <xacro:get_visual_params name="wrist_3" type="visual_offset"/>
+      <xacro:get_visual_params name="wrist_3" type="visual_offset"/>
       <visual>
         <origin xyz="0 0 ${visual_params}" rpy="${pi/2} 0 0"/>
@@ -258,5 +195,5 @@
         </geometry>
       </collision>
-      <xacro:cylinder_inertial radius="${wrist_3_inertia_radius}" length="${wrist_3_inertia_length}"  mass="${wrist_3_mass}">
+      <xacro:cylinder_inertial radius="${wrist_3_inertia_radius}" length="${wrist_3_inertia_length}" mass="${wrist_3_mass}">
         <origin xyz="0.0 0.0 ${-0.5 * wrist_3_inertia_length}" rpy="0 0 0" />
       </xacro:cylinder_inertial>
@@ -265,5 +202,5 @@
     <link name="base_table">
       <visual>
-        <origin xyz="0 0 0.25" />
+        <origin xyz="0 0 0.0" />
         <geometry>
           <box size="1.32 0.8 0.5" />
@@ -272,5 +209,5 @@
       </visual>
       <collision>
-        <origin xyz="0 0 0.25" />
+        <origin xyz="0 0 0.0" />
         <geometry>
           <box size="1.32 0.8 0.5" />
@@ -280,14 +217,104 @@
     <link name="profile1">
       <visual>
-      <origin xyz="0 0 0.45" />
-        <geometry>
-          <box size="0.03 0.35 0.9" />
+        <origin xyz="0 0 0" />
+        <geometry>
+          <box size="0.04 0.35 0.9" />
         </geometry>
         <material name="blue" />
       </visual>
       <collision>
-        <origin xyz="0 0 0.45" />
-        <geometry>
-          <box size="0.03 0.35 0.9" />
+        <origin xyz="0 0 0" />
+        <geometry>
+          <box size="0.04 0.35 0.9" />
+        </geometry>
+      </collision>
+    </link>
+    <link name="wall1">
+      <visual>
+        <origin xyz="0 0 0" />
+        <geometry>
+          <box size="0.06 0.8 0.25" />
+        </geometry>
+        <material name="blue" />
+      </visual>
+      <collision>
+        <origin xyz="0 0 0" />
+        <geometry>
+          <box size="0.06 0.8 0.25" />
+        </geometry>
+      </collision>
+    </link>
+    <link name="wall2">
+      <visual>
+        <origin xyz="0 0 0" />
+        <geometry>
+          <box size="1.32 0.06 0.5" />
+        </geometry>
+        <material name="blue" />
+      </visual>
+      <collision>
+        <origin xyz="0 0 0" />
+        <geometry>
+          <box size="1.32 0.06 0.5" />
+        </geometry>
+      </collision>
+    </link>
+    <link name="box1">
+      <visual>
+        <origin xyz="0 0 0" />
+        <geometry>
+          <box size="0.015 0.44 0.20" />
+        </geometry>
+        <material name="orange" />
+      </visual>
+      <collision>
+        <origin xyz="0 0 0" />
+        <geometry>
+          <box size="0.015 0.44 0.20" />
+        </geometry>
+      </collision>
+    </link>
+    <link name="box2">
+      <visual>
+        <origin xyz="0 0 0" />
+        <geometry>
+          <box size="0.015 0.44 0.20" />
+        </geometry>
+        <material name="orange" />
+      </visual>
+      <collision>
+        <origin xyz="0 0 0" />
+        <geometry>
+          <box size="0.015 0.44 0.20" />
+        </geometry>
+      </collision>
+    </link>
+    <link name="box3">
+      <visual>
+        <origin xyz="0 0 0" />
+        <geometry>
+          <box size="0.24 0.015 0.20" />
+        </geometry>
+        <material name="orange" />
+      </visual>
+      <collision>
+        <origin xyz="0 0 0" />
+        <geometry>
+          <box size="0.24 0.015 0.20" />
+        </geometry>
+      </collision>
+    </link>
+    <link name="box4">
+      <visual>
+        <origin xyz="0 0 0" />
+        <geometry>
+          <box size="0.24 0.015 0.20" />
+        </geometry>
+        <material name="orange" />
+      </visual>
+      <collision>
+        <origin xyz="0 0 0" />
+        <geometry>
+          <box size="0.24 0.015 0.20" />
         </geometry>
       </collision>
@@ -295,16 +322,46 @@
     <!-- Define my joint -->
     <joint name="{tf_prefix}base_table_joint" type="fixed">
-      <origin xyz="0 0 0" rpy="0 0 0"/>
+      <origin xyz="0 0 ${-0.25 + gazebo_axis_z}" rpy="0 0 0"/>
       <parent link="${parent}" />
       <child link="base_table" />
     </joint>
     <joint name="${tf_prefix}profile_joint" type="fixed">
-      <origin xyz="0.3 0 0.505" rpy="0 0 0"/>
+      <origin xyz="0.53 0 0.701" rpy="0 0 0"/>
       <parent link="base_table" />
       <child link="profile1" />
+    </joint>
+    <joint name="${tf_prefix}wall1_joint" type="fixed">
+      <origin xyz="-0.695 0 0.375" rpy="0 0 0"/>
+      <parent link="base_table" />
+      <child link="wall1" />
+    </joint>
+    <joint name="${tf_prefix}wall2_joint" type="fixed">
+      <origin xyz="0 -0.415 0.51" rpy="0 0 0"/>
+      <parent link="base_table" />
+      <child link="wall2" />
+    </joint>
+    <joint name="${tf_prefix}box1_joint" type="fixed">
+      <origin xyz="-0.295 0.0 0.351" rpy="0 0 0"/>
+      <parent link="base_table" />
+      <child link="box1" />
+    </joint>
+    <joint name="${tf_prefix}box2_joint" type="fixed">
+      <origin xyz="-0.535 0.0 0.351" rpy="0 0 0"/>
+      <parent link="base_table" />
+      <child link="box2" />
+    </joint>
+    <joint name="${tf_prefix}box3_joint" type="fixed">
+      <origin xyz="-0.415 -0.2285 0.351" rpy="0 0 0"/>
+      <parent link="base_table" />
+      <child link="box3" />
+    </joint>
+    <joint name="${tf_prefix}box4_joint" type="fixed">
+      <origin xyz="-0.415 0.2285 0.351" rpy="0 0 0"/>
+      <parent link="base_table" />
+      <child link="box4" />
     </joint>
     <!-- base_joint fixes base_link to the environment -->
     <joint name="${tf_prefix}base_joint" type="fixed">
-      <origin xyz="0 0 0.505" rpy="0 0 0"/>
+      <origin xyz="0 0 0.251" rpy="0 0 0"/>
       <xacro:insert_block name="origin" />
       <parent link="base_table" />
@@ -327,8 +384,7 @@
       <origin xyz="${shoulder_x} ${shoulder_y} ${shoulder_z}" rpy="${shoulder_roll} ${shoulder_pitch} ${shoulder_yaw}" />
       <axis xyz="0 0 1" />
-      <limit lower="${shoulder_pan_lower_limit}" upper="${shoulder_pan_upper_limit}"
-        effort="${shoulder_pan_effort_limit}" velocity="${shoulder_pan_velocity_limit}"/>
-      <xacro:if value="${safety_limits}">
-         <safety_controller soft_lower_limit="${shoulder_pan_lower_limit + safety_pos_margin}" soft_upper_limit="${shoulder_pan_upper_limit - safety_pos_margin}" k_position="${safety_k_position}" k_velocity="0.0"/>
+      <limit lower="${shoulder_pan_lower_limit}" upper="${shoulder_pan_upper_limit}" effort="${shoulder_pan_effort_limit}" velocity="${shoulder_pan_velocity_limit}"/>
+      <xacro:if value="${safety_limits}">
+        <safety_controller soft_lower_limit="${shoulder_pan_lower_limit + safety_pos_margin}" soft_upper_limit="${shoulder_pan_upper_limit - safety_pos_margin}" k_position="${safety_k_position}" k_velocity="0.0"/>
       </xacro:if>
       <dynamics damping="0" friction="0"/>
@@ -339,8 +395,7 @@
       <origin xyz="${upper_arm_x} ${upper_arm_y} ${upper_arm_z}" rpy="${upper_arm_roll} ${upper_arm_pitch} ${upper_arm_yaw}" />
       <axis xyz="0 0 1" />
-      <limit lower="${shoulder_lift_lower_limit}" upper="${shoulder_lift_upper_limit}"
-        effort="${shoulder_lift_effort_limit}" velocity="${shoulder_lift_velocity_limit}"/>
-      <xacro:if value="${safety_limits}">
-         <safety_controller soft_lower_limit="${shoulder_lift_lower_limit + safety_pos_margin}" soft_upper_limit="${shoulder_lift_upper_limit - safety_pos_margin}" k_position="${safety_k_position}" k_velocity="0.0"/>
+      <limit lower="${shoulder_lift_lower_limit}" upper="${shoulder_lift_upper_limit}" effort="${shoulder_lift_effort_limit}" velocity="${shoulder_lift_velocity_limit}"/>
+      <xacro:if value="${safety_limits}">
+        <safety_controller soft_lower_limit="${shoulder_lift_lower_limit + safety_pos_margin}" soft_upper_limit="${shoulder_lift_upper_limit - safety_pos_margin}" k_position="${safety_k_position}" k_velocity="0.0"/>
       </xacro:if>
       <dynamics damping="0" friction="0"/>
@@ -351,8 +406,7 @@
       <origin xyz="${forearm_x} ${forearm_y} ${forearm_z}" rpy="${forearm_roll} ${forearm_pitch} ${forearm_yaw}" />
       <axis xyz="0 0 1" />
-      <limit lower="${elbow_joint_lower_limit}" upper="${elbow_joint_upper_limit}"
-        effort="${elbow_joint_effort_limit}" velocity="${elbow_joint_velocity_limit}"/>
-      <xacro:if value="${safety_limits}">
-         <safety_controller soft_lower_limit="${elbow_joint_lower_limit + safety_pos_margin}" soft_upper_limit="${elbow_joint_upper_limit - safety_pos_margin}" k_position="${safety_k_position}" k_velocity="0.0"/>
+      <limit lower="${elbow_joint_lower_limit}" upper="${elbow_joint_upper_limit}" effort="${elbow_joint_effort_limit}" velocity="${elbow_joint_velocity_limit}"/>
+      <xacro:if value="${safety_limits}">
+        <safety_controller soft_lower_limit="${elbow_joint_lower_limit + safety_pos_margin}" soft_upper_limit="${elbow_joint_upper_limit - safety_pos_margin}" k_position="${safety_k_position}" k_velocity="0.0"/>
       </xacro:if>
       <dynamics damping="0" friction="0"/>
@@ -363,8 +417,7 @@
       <origin xyz="${wrist_1_x} ${wrist_1_y} ${wrist_1_z}" rpy="${wrist_1_roll} ${wrist_1_pitch} ${wrist_1_yaw}" />
       <axis xyz="0 0 1" />
-      <limit lower="${wrist_1_lower_limit}" upper="${wrist_1_upper_limit}"
-        effort="${wrist_1_effort_limit}" velocity="${wrist_1_velocity_limit}"/>
-      <xacro:if value="${safety_limits}">
-         <safety_controller soft_lower_limit="${wrist_1_lower_limit + safety_pos_margin}" soft_upper_limit="${wrist_1_upper_limit - safety_pos_margin}" k_position="${safety_k_position}" k_velocity="0.0"/>
+      <limit lower="${wrist_1_lower_limit}" upper="${wrist_1_upper_limit}" effort="${wrist_1_effort_limit}" velocity="${wrist_1_velocity_limit}"/>
+      <xacro:if value="${safety_limits}">
+        <safety_controller soft_lower_limit="${wrist_1_lower_limit + safety_pos_margin}" soft_upper_limit="${wrist_1_upper_limit - safety_pos_margin}" k_position="${safety_k_position}" k_velocity="0.0"/>
       </xacro:if>
       <dynamics damping="0" friction="0"/>
@@ -375,8 +428,7 @@
       <origin xyz="${wrist_2_x} ${wrist_2_y} ${wrist_2_z}" rpy="${wrist_2_roll} ${wrist_2_pitch} ${wrist_2_yaw}" />
       <axis xyz="0 0 1" />
-      <limit lower="${wrist_2_lower_limit}" upper="${wrist_2_upper_limit}"
-             effort="${wrist_2_effort_limit}" velocity="${wrist_2_velocity_limit}"/>
-      <xacro:if value="${safety_limits}">
-         <safety_controller soft_lower_limit="${wrist_2_lower_limit + safety_pos_margin}" soft_upper_limit="${wrist_2_upper_limit - safety_pos_margin}" k_position="${safety_k_position}" k_velocity="0.0"/>
+      <limit lower="${wrist_2_lower_limit}" upper="${wrist_2_upper_limit}" effort="${wrist_2_effort_limit}" velocity="${wrist_2_velocity_limit}"/>
+      <xacro:if value="${safety_limits}">
+        <safety_controller soft_lower_limit="${wrist_2_lower_limit + safety_pos_margin}" soft_upper_limit="${wrist_2_upper_limit - safety_pos_margin}" k_position="${safety_k_position}" k_velocity="0.0"/>
       </xacro:if>
       <dynamics damping="0" friction="0"/>
@@ -387,8 +439,7 @@
       <origin xyz="${wrist_3_x} ${wrist_3_y} ${wrist_3_z}" rpy="${wrist_3_roll} ${wrist_3_pitch} ${wrist_3_yaw}" />
       <axis xyz="0 0 1" />
-      <limit lower="${wrist_3_lower_limit}" upper="${wrist_3_upper_limit}"
-             effort="${wrist_3_effort_limit}" velocity="${wrist_3_velocity_limit}"/>
-      <xacro:if value="${safety_limits}">
-         <safety_controller soft_lower_limit="${wrist_3_lower_limit + safety_pos_margin}" soft_upper_limit="${wrist_3_upper_limit - safety_pos_margin}" k_position="${safety_k_position}" k_velocity="0.0"/>
+      <limit lower="${wrist_3_lower_limit}" upper="${wrist_3_upper_limit}" effort="${wrist_3_effort_limit}" velocity="${wrist_3_velocity_limit}"/>
+      <xacro:if value="${safety_limits}">
+        <safety_controller soft_lower_limit="${wrist_3_lower_limit + safety_pos_margin}" soft_upper_limit="${wrist_3_upper_limit - safety_pos_margin}" k_position="${safety_k_position}" k_velocity="0.0"/>
       </xacro:if>
       <dynamics damping="0" friction="0"/>
@@ -427,4 +478,10 @@
       <child link="${tf_prefix}tool0"/>
     </joint>
+    <link name="${tf_prefix}ee_link" />
+    <joint name="gripper_joint" type="fixed">
+      <origin xyz="0 0 0.215" rpy="0 0 0" />
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